Commit message: Modified folder references

File: urdf/licas/licasa1_testbench.urdf.xacro (robot description, xacro)
@@ -3,8 +3,8 @@
 <robot name="LiCAS_A1" xmlns:xacro="http://ros.org/wiki/xacro">
 <!-- Import Transmissions -->
-<xacro:include filename="$(find licasa1_description)/urdf/licasa1_testbench.transmission.xacro" />
+<xacro:include filename="$(find cable_suspended_robotics)/urdf/licas/licasa1_testbench.transmission.xacro" />
 <xacro:LiCAS_A1_transmission name="LiCAS_A1" hardware_interface1="hardware_interface/PositionJointInterface" hardware_interface2="hardware_interface/EffortJointInterface" />
 <!-- Import Gazebo plugins -->
-<xacro:include filename="$(find licasa1_description)/gazebo/gazebo.urdf.xacro"/>
+<xacro:include filename="$(find cable_suspended_robotics)/gazebo/licas/gazebo.urdf.xacro"/>
 <link name="world"/>
 <!-- TESTBENCH -->
@@ -124,11 +124,11 @@
     <origin xyz="0 0 0"/>
     <geometry>
-      <mesh filename="package://licasa1_description/mesh/Shoulder_Pitch_Structure.dae" scale=".001 .001 .001"/>
-    </geometry>
-  </visual>
-  <collision>
-    <origin xyz="0 0 0"/>
-    <geometry>
-      <mesh filename="package://licasa1_description/mesh/Shoulder_Pitch_Structure.dae" scale=".001 .001 .001"/>
+      <mesh filename="package://cable_suspended_robotics/mesh/licas/Shoulder_Pitch_Structure.dae" scale=".001 .001 .001"/>
+    </geometry>
+  </visual>
+  <collision>
+    <origin xyz="0 0 0"/>
+    <geometry>
+      <mesh filename="package://cable_suspended_robotics/mesh/licas/Shoulder_Pitch_Structure.dae" scale=".001 .001 .001"/>
     </geometry>
   </collision>
@@ -152,5 +152,5 @@
     <origin xyz="0 0.04 0"/>
     <geometry>
-      <mesh filename="package://licasa1_description/mesh/Shoulder_Roll_Structure_Left.dae" scale=".001 .001 .001"/>
+      <mesh filename="package://cable_suspended_robotics/mesh/licas/Shoulder_Roll_Structure_Left.dae" scale=".001 .001 .001"/>
     </geometry>
   </visual>
@@ -158,5 +158,5 @@
     <origin xyz="0 0.04 0"/>
     <geometry>
-      <mesh filename="package://licasa1_description/mesh/Shoulder_Roll_Structure_Left.dae" scale=".001 .001 .001"/>
+      <mesh filename="package://cable_suspended_robotics/mesh/licas/Shoulder_Roll_Structure_Left.dae" scale=".001 .001 .001"/>
     </geometry>
   </collision>
@@ -179,11 +179,11 @@
     <origin xyz="0 0 0"/>
     <geometry>
-      <mesh filename="package://licasa1_description/mesh/Assembly_Shoulder_Yaw_Structure.dae" scale=".001 .001 .001"/>
-    </geometry>
-  </visual>
-  <collision>
-    <origin xyz="0 0 0"/>
-    <geometry>
-      <mesh filename="package://licasa1_description/mesh/Assembly_Shoulder_Yaw_Structure.dae" scale=".001 .001 .001"/>
+      <mesh filename="package://cable_suspended_robotics/mesh/licas/Assembly_Shoulder_Yaw_Structure.dae" scale=".001 .001 .001"/>
+    </geometry>
+  </visual>
+  <collision>
+    <origin xyz="0 0 0"/>
+    <geometry>
+      <mesh filename="package://cable_suspended_robotics/mesh/licas/Assembly_Shoulder_Yaw_Structure.dae" scale=".001 .001 .001"/>
     </geometry>
   </collision>
@@ -206,5 +206,5 @@
     <origin xyz="0 0 -0.132"/>
     <geometry>
-      <mesh filename="package://licasa1_description/mesh/Elbow_Pitch_Structure_Left_Cut.dae" scale=".001 .001 .001"/>
+      <mesh filename="package://cable_suspended_robotics/mesh/licas/Elbow_Pitch_Structure_Left_Cut.dae" scale=".001 .001 .001"/>
     </geometry>
   </visual>
@@ -212,5 +212,5 @@
     <origin xyz="0 0 -0.132"/>
     <geometry>
-      <mesh filename="package://licasa1_description/mesh/Elbow_Pitch_Structure_Left_Cut.dae" scale=".001 .001 .001"/>
+      <mesh filename="package://cable_suspended_robotics/mesh/licas/Elbow_Pitch_Structure_Left_Cut.dae" scale=".001 .001 .001"/>
     </geometry>
   </collision>
@@ -233,11 +233,11 @@
     <origin xyz="0 0 0"/>
     <geometry>
-      <mesh filename="package://licasa1_description/mesh/Forearm_Link_with_Gripper_Servo.dae" scale=".001 .001 .001"/>
-    </geometry>
-  </visual>
-  <collision>
-    <origin xyz="0 0 0"/>
-    <geometry>
-      <mesh filename="package://licasa1_description/mesh/Forearm_Link_with_Gripper_Servo.dae" scale=".001 .001 .001"/>
+      <mesh filename="package://cable_suspended_robotics/mesh/licas/Forearm_Link_with_Gripper_Servo.dae" scale=".001 .001 .001"/>
+    </geometry>
+  </visual>
+  <collision>
+    <origin xyz="0 0 0"/>
+    <geometry>
+      <mesh filename="package://cable_suspended_robotics/mesh/licas/Forearm_Link_with_Gripper_Servo.dae" scale=".001 .001 .001"/>
     </geometry>
   </collision>
@@ -261,5 +261,5 @@
     <origin xyz="0 -0.04 0"/>
     <geometry>
-      <mesh filename="package://licasa1_description/mesh/Shoulder_Roll_Structure_Right.dae" scale=".001 .001 .001"/>
+      <mesh filename="package://cable_suspended_robotics/mesh/licas/Shoulder_Roll_Structure_Right.dae" scale=".001 .001 .001"/>
     </geometry>
   </visual>
@@ -267,5 +267,5 @@
     <origin xyz="0 -0.04 0"/>
     <geometry>
-      <mesh filename="package://licasa1_description/mesh/Shoulder_Roll_Structure_Right.dae" scale=".001 .001 .001"/>
+      <mesh filename="package://cable_suspended_robotics/mesh/licas/Shoulder_Roll_Structure_Right.dae" scale=".001 .001 .001"/>
     </geometry>
   </collision>
@@ -288,11 +288,11 @@
     <origin xyz="0 0 0"/>
     <geometry>
-      <mesh filename="package://licasa1_description/mesh/Assembly_Shoulder_Yaw_Structure.dae" scale=".001 .001 .001"/>
-    </geometry>
-  </visual>
-  <collision>
-    <origin xyz="0 0 0"/>
-    <geometry>
-      <mesh filename="package://licasa1_description/mesh/Assembly_Shoulder_Yaw_Structure.dae" scale=".001 .001 .001"/>
+      <mesh filename="package://cable_suspended_robotics/mesh/licas/Assembly_Shoulder_Yaw_Structure.dae" scale=".001 .001 .001"/>
+    </geometry>
+  </visual>
+  <collision>
+    <origin xyz="0 0 0"/>
+    <geometry>
+      <mesh filename="package://cable_suspended_robotics/mesh/licas/Assembly_Shoulder_Yaw_Structure.dae" scale=".001 .001 .001"/>
     </geometry>
   </collision>
@@ -315,5 +315,5 @@
     <origin xyz="0 0 -0.132"/>
     <geometry>
-      <mesh filename="package://licasa1_description/mesh/Elbow_Pitch_Structure_Right_Cut.dae" scale=".001 .001 .001"/>
+      <mesh filename="package://cable_suspended_robotics/mesh/licas/Elbow_Pitch_Structure_Right_Cut.dae" scale=".001 .001 .001"/>
     </geometry>
   </visual>
@@ -321,5 +321,5 @@
     <origin xyz="0 0 -0.132"/>
     <geometry>
-      <mesh filename="package://licasa1_description/mesh/Elbow_Pitch_Structure_Right_Cut.dae" scale=".001 .001 .001"/>
+      <mesh filename="package://cable_suspended_robotics/mesh/licas/Elbow_Pitch_Structure_Right_Cut.dae" scale=".001 .001 .001"/>
     </geometry>
   </collision>
@@ -342,11 +342,11 @@
     <origin xyz="0 0 0"/>
     <geometry>
-      <mesh filename="package://licasa1_description/mesh/Forearm_Link_with_Gripper_Servo.dae" scale=".001 .001 .001"/>
-    </geometry>
-  </visual>
-  <collision>
-    <origin xyz="0 0 0"/>
-    <geometry>
-      <mesh filename="package://licasa1_description/mesh/Forearm_Link_with_Gripper_Servo.dae" scale=".001 .001 .001"/>
+      <mesh filename="package://cable_suspended_robotics/mesh/licas/Forearm_Link_with_Gripper_Servo.dae" scale=".001 .001 .001"/>
+    </geometry>
+  </visual>
+  <collision>
+    <origin xyz="0 0 0"/>
+    <geometry>
+      <mesh filename="package://cable_suspended_robotics/mesh/licas/Forearm_Link_with_Gripper_Servo.dae" scale=".001 .001 .001"/>
     </geometry>
   </collision>
